File: doc/Sagetech-ardu.sch (KiCad schematic (older format))
At the start: 5 parts

Commit message: Updated schematic
Parts:
- renumbered RS232 to RS232~LEVEL~SHIFTER
Changed lines of the file:
@@
 Sheet 1 1
 Title "Sagetech ADSB Transponder integration with Ardupilot"
-Date "11 feb 2015"
+Date "17 feb 2015"
 Rev ""
 Comp ""
@@
 23444
 $Comp
-L CONVERTER232 RS232
+L CONVERTER232 RS232~LEVEL~SHIFTER
 U 1 1 54BF8AAA
 P 6050 5500
-F 0 "RS232" H 6300 4650 60  0000 C CNN
+F 0 "RS232 LEVEL SHIFTER" H 6300 4650 60  0000 C CNN
 F 1 "CONVERTER232" H 6250 5550 60  0001 C CNN
 F 2 "" H 6100 5500 60  0000 C CNN
